File: body.kicad_pcb (KiCad board)
At the start: 2 copper layers, 37.5 x 50.8 mm, 35 parts, among them P1 CON_VIN, P13 CON_STEP, P14 CON_SRV_CAM, P15 CON_SRV_BRAKE, P16 CON_SRV_LOCK, P17 CON_POLOLU_DRV8834, P18 CON_BAT, P19 CON_UART, P2 CON_FAN2, P20 CON_STEP_STOP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

Commit message: Updated design
Parts:
- removed P2: CON_FAN2, Connectors_Molex:Molex_PicoBlade_53261-0371
- added P3: CON_I2C, Connectors_Molex:Molex_PicoBlade_53047-0210, B.Cu at (165.1, 111.8)
- added P4: CON_LED, Connectors_Molex:Molex_PicoBlade_53047-0410, B.Cu at (147.3, 95.2)
- P20: footprint Connectors_Molex:Molex_PicoBlade_53047-0210 -> Connectors_Molex:Molex_PicoBlade_53047-0310
- U14: value FOOT_SWITCH -> LED_SWITCH
- moved P20 24.2 mm to (157.5, 110.5)
- moved U8 15.3 mm to (149.9, 102.7)
- moved C3 15.3 mm to (150.6, 105.4)
- moved P16 11.4 mm to (152.4, 90.2)
- moved P23 8.93 mm to (162.6, 90.2)
- moved P14 8.85 mm to (155.0, 94.0)
- moved P15 7.73 mm to (162.6, 94.0)
- moved C6 3.81 mm to (158.0, 119.4)
- moved U13 3.49 mm to (158.6, 121.6)
- moved P26 2.82 mm to (156.2, 87.6), turned to 180 degrees
- moved C7 1.80 mm to (146.6, 105.4)
- moved U14 1.80 mm to (146.1, 102.9)
- moved C5 1.77 mm to (155.2, 106.5), turned to 180 degrees
- moved P1 1.29 mm to (166.4, 107.9)
- moved P18 1.27 mm to (166.4, 102.9)
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Connections:
- net /BAT_STAT1 renamed /BAT1_STAT
- net /BAT_STAT2 renamed /BAT2_STAT
- P19 pad 2: /RXD -> /TXD
- P19 pad 3: /TXD -> /RXD
- P19 pad 4: VCC -> /HOST_INT
- P20 pad 1: /STEP_STOP -> /STEP_STOP1
- P20 pad 2: GND -> /STEP_STOP2
- P23 pad 2: /FOOT_VOUT -> /SRV_VOUT
- P24 pad 1: /EP_RXD -> GND
- P24 pad 2: /EP_TXD -> /FRAME_STOP
- P24 pad 3: /FRAME_STOP -> /EP_TXD
- P24 pad 4: GND -> /EP_RXD
- U10 pad 21: /FAN_TACHO -> /EP_EN
- U10 pad 22: /EP_EN -> /LED_EN
- U10 pad 23: /FOOT_EN -> /FRAME_STOP
- U10 pad 24: /TMP_EN -> /STEP_STOP1
- U10 pad 25: /SRV_EN -> /STEP_STOP2
- U10 pad 26: (no net) -> /SRV_EN
- U10 pad 27: (no net) -> /FAN_EN
- U10 pad 28: (no net) -> /FAN_TACHO
- U10 pad 4: /STEP_STOP -> /~STEP_SLP
- U10 pad 5: /FRAME_STOP -> /HOST_INT
- U11 pad 18: /~STEP_SLP -> /LED_DAT
- U11 pad 19: /TMP -> /LED_CLK
- U11 pad 20: /~IO_RST -> /TMP
- U11 pad 9: /FAN_EN -> /~IO_RST
- U12 pad 5: /TXD -> /RXD
- U12 pad 6: /RXD -> /TXD
- U14 pad 1: /FOOT_VOUT -> /LED_VOUT
- U14 pad 4: /FOOT_EN -> /LED_EN
- U16 pad 4: /TMP_EN -> VCC
Routing:
- net /HOST_INT: track 0.00 -> 72.0 mm, vias 0 -> 1
- net /STEP_STOP: track 46.1 -> 0.00 mm
- net VCC: track 115.8 -> 159.2 mm
- net /TMP_EN: track 39.3 -> 0.00 mm, vias 2 -> 0
- net /FOOT_EN: track 30.9 -> 0.00 mm, vias 2 -> 0
- net /LED_EN: track 0.00 -> 30.3 mm, vias 0 -> 2
- net /SRV_EN: track 56.7 -> 30.9 mm, vias 0 -> 2
- net /~IO_RST: track 32.8 -> 9.11 mm
- net /STEP_STOP2: track 0.00 -> 22.8 mm, vias 0 -> 1
- net /STEP_STOP1: track 0.00 -> 20.2 mm
- net /FOOT_VOUT: track 16.3 -> 0.00 mm, vias 1 -> 0
- net /~STEP_SLP: track 14.6 -> 30.2 mm, vias 0 -> 1
- net /SRV_VOUT: track 15.7 -> 31.1 mm
- net /FAN_VOUT: track 22.7 -> 11.1 mm
- net /FRAME_STOP: track 49.5 -> 38.0 mm
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